File: WT_S32M2_EVB.kicad_sch (KiCad schematic)
At the start: 0 parts

Commit message: Update
Other:
- sheet JTAG ports: added DBG, TCK, TDI, TDO, TMS; removed SWCLK, SWDIO, SWO
- sheet MCU ports: added DBG, TCK, TDI, TDO, TMS; removed SWCLK, SWDIO, SWO
Changed lines of the file:
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@@
+	(wire
+		(pts
+			(xy 121.92 88.9) (xy 133.35 88.9)
+		)
+		(stroke
+			(width 0)
+			(type default)
+		)
+	)
+	(wire
+		(pts
+			(xy 121.92 96.52) (xy 133.35 96.52)
+		)
+		(stroke
+			(width 0)
+			(type default)
+		)
+	)
 	(wire
 		(pts
@@
 	(wire
 		(pts
+			(xy 121.92 91.44) (xy 133.35 91.44)
+		)
+		(stroke
+			(width 0)
+			(type default)
+		)
+	)
+	(wire
+		(pts
 			(xy 121.92 93.98) (xy 133.35 93.98)
 		)
@@
 	(wire
 		(pts
-			(xy 121.92 88.9) (xy 133.35 88.9)
-		)
-		(stroke
-			(width 0)
-			(type default)
-		)
-	)
-	(wire
-		(pts
-			(xy 121.92 91.44) (xy 133.35 91.44)
+			(xy 121.92 83.82) (xy 133.35 83.82)
 		)
 		(stroke
@@
 			)
 		)
-		(pin "SWCLK" output
-			(at 121.92 88.9 0)
+		(pin "DBG" input
+			(at 121.92 96.52 0)
+			(effects
+				(font
+					(size 1.27 1.27)
+				)
+				(justify right)
+			)
+		)
+		(pin "TCK" output
+			(at 121.92 86.36 0)
+			(effects
+				(font
+					(size 1.27 1.27)
+				)
+				(justify right)
+			)
+		)
+		(pin "TMS" bidirectional
+			(at 121.92 83.82 0)
+			(effects
+				(font
+					(size 1.27 1.27)
+				)
+				(justify right)
+			)
+		)
+		(pin "TDO" output
+			(at 121.92 91.44 0)
 			(effects
 				(font
@@
 			)
 		)
-		(pin "SWO" input
-			(at 121.92 91.44 0)
-			(effects
-				(font
-					(size 1.27 1.27)
-				)
-				(justify right)
-			)
-		)
-		(pin "SWDIO" bidirectional
-			(at 121.92 86.36 0)
+		(pin "TDI" input
+			(at 121.92 88.9 0)
 			(effects
 				(font
@@
 			)
 		)
-		(pin "SWCLK" input
-			(at 133.35 88.9 180)
-			(effects
-				(font
-					(size 1.27 1.27)
-				)
-				(justify left)
-			)
-		)
-		(pin "SWO" output
-			(at 133.35 91.44 180)
-			(effects
-				(font
-					(size 1.27 1.27)
-				)
-				(justify left)
-			)
-		)
-		(pin "SWDIO" bidirectional
-			(at 133.35 86.36 180)
+		(pin "DBG" output
+			(at 133.35 96.52 180)
 			(effects
 				(font
@@
 			(effects
 				(font
+					(size 1.27 1.27)
+				)
+				(justify left)
+			)
+		)
+		(pin "TDI" output
+			(at 133.35 88.9 180)
+			(effects
+				(font
+					(size 1.27 1.27)
+				)
+				(justify left)
+			)
+		)
+		(pin "TDO" input
+			(at 133.35 91.44 180)
+			(effects
+				(font
+					(size 1.27 1.27)
+				)
+				(justify left)
+			)
+		)
+		(pin "TCK" input
+			(at 133.35 86.36 180)
+			(effects
+				(font
+					(size 1.27 1.27)
+				)
+				(justify left)
+			)
+		)
+		(pin "TMS" bidirectional
+			(at 133.35 83.82 180)
+			(effects
+				(font
