File: mcu.kicad_sch (KiCad schematic)
At the start: 7 parts, among them J3 Conn_01x16_Pin, J4 Conn_01x16_Pin, J5 Conn_01x16_Pin, J6 Conn_01x16_Pin, SW1 KEY

Commit message: Update
Parts:
- added C10, C7: 12p, Capacitor_SMD:C_0805_2012Metric, symbol Device:C
- added R6, R7: 0, Resistor_SMD:R_0805_2012Metric, symbol Device:R
- added U2: S32M242CCABMKHST, Package_QFP:LQFP-64-1EP_10x10mm_P0.5mm_EP6.5x6.5mm_ThermalVias, symbol MCU_NXP_S32M2:S32M242CCABMKHST
- added Y1: 8M, Crystal:Crystal_HC49-4H_Vertical, symbol Device:Crystal
Connections:
- net GNDD: now also C10.2, C7.2
- net RESET: now also J6.14 (Pin_14), U2.46 (RESET_B)
- net PIN49: now reaches J4.1 (Pin_1)
- net PIN49: now also U2.49 (LS0)
- net PIN58: now reaches J4.10 (Pin_10)
- net PIN58: now also U2.58 (LS1)
- net PIN59: now reaches J4.11 (Pin_11)
- net PIN59: now also U2.59 (LS2)
- net PIN60: now reaches J4.12 (Pin_12)
- net PIN60: now also U2.60 (LG2)
- net PIN61: now reaches J4.13 (Pin_13)
- net PIN61: now also U2.61 (HS2)
- net PIN62: now reaches J4.14 (Pin_14)
- net PIN62: now also U2.62 (HG2)
- net PIN63: now reaches J4.15 (Pin_15)
- net PIN63: now also U2.63 (VBS2)
- net PIN64: now reaches J4.16 (Pin_16)
- net PIN64: now also U2.64 (VCP)
- net PIN50: now reaches J4.2 (Pin_2)
- net PIN50: now also U2.50 (LG0)
- net PIN51: now reaches J4.3 (Pin_3)
- net PIN51: now also U2.51 (HS0)
- net PIN52: now reaches J4.4 (Pin_4)
- net PIN52: now also U2.52 (HG0)
- net PIN53: now reaches J4.5 (Pin_5)
- net PIN53: now also U2.53 (VBS0)
- net PIN54: now reaches J4.6 (Pin_6)
- net PIN54: now also U2.54 (VBS1)
- net PIN55: now reaches J4.7 (Pin_7)
- net PIN55: now also U2.55 (HG1)
- net PIN56: now reaches J4.8 (Pin_8)
- net PIN56: now also U2.56 (HS1)
- net PIN57: now reaches J4.9 (Pin_9)
- net PIN57: now also U2.57 (LG1)
- net TMS: now reaches J5.1 (Pin_1)
- net TMS: now also U2.17 (PTA4)
- net PIN26: now reaches J5.10 (Pin_10)
- net PIN27: now reaches J5.11 (Pin_11)
- net PIN28: now reaches J5.12 (Pin_12)
- net PIN29: now reaches J5.13 (Pin_13)
- net PIN29: now also R7.1, U2.29 (PTB7)
- net PIN30: now reaches J5.14 (Pin_14)
- net PIN30: now also R6.1, U2.30 (PTB6)
- net PIN31: now reaches J5.15 (Pin_15)
- net PIN31: now also U2.31 (PTD16)
- net PIN32: now reaches J5.16 (Pin_16)
- net PIN32: now also U2.32 (PTD15)
- net PIN18: now reaches J5.2 (Pin_2)
- net PIN18: now also U2.18 (PTE16)
- net PIN19: now reaches J5.3 (Pin_3)
- net PIN19: now also U2.19 (PTE15)
- net PIN20: now reaches J5.4 (Pin_4)
- net PIN20: now also U2.20 (PTD1)
- net PIN21: now reaches J5.5 (Pin_5)
- net PIN21: now also U2.21 (PTD0)
- net PIN22: now reaches J5.6 (Pin_6)
- net PIN22: now also U2.22 (PTE11)
- net PIN23: now reaches J5.7 (Pin_7)
- net PIN23: now also U2.23 (PTE5)
- net PIN24: now reaches J5.8 (Pin_8)
- net PIN24: now also U2.24 (PTE4)
- net PIN25: now reaches J5.9 (Pin_9)
- net PIN33: now reaches J6.1 (Pin_1)
- net PIN33: now also U2.33 (PTB5)
- net PIN42: now reaches J6.10 (Pin_10)
- net PIN42: now also U2.42 (VDDC)
- net PIN43: now reaches J6.11 (Pin_11)
- net PIN43: now also U2.43 (HVI)
- net PIN44: now reaches J6.12 (Pin_12)
- net PIN44: now also U2.44 (AMPM)
- net PIN45: now reaches J6.13 (Pin_13)
- net PIN45: now also U2.45 (AMPP)
- net PIN47: now reaches J6.15 (Pin_15)
- net PIN47: now also U2.47 (AMPOUT)
- net PIN48: now reaches J6.16 (Pin_16)
- net PIN34: now reaches J6.2 (Pin_2)
- net PIN34: now also U2.34 (PTB4)
- net DBG: now reaches J6.3 (Pin_3)
- net DBG: now also U2.35 (PTC3)
- net PIN36: now reaches J6.4 (Pin_4)
- net PIN36: now also U2.36 (PTC2)
- net PIN37: now reaches J6.5 (Pin_5)
- net PIN37: now also U2.37 (PTC1)
- net PIN38: now reaches J6.6 (Pin_6)
- net PIN38: now also U2.38 (PTC0)
- net PIN39: now reaches J6.7 (Pin_7)
- net PIN39: now also U2.39 (VSSC)
- net PIN40: now reaches J6.8 (Pin_8)
- net PIN40: now also U2.40 (CANL)
- net PIN41: now reaches J6.9 (Pin_9)
- net PIN41: now also U2.41 (CANH)
- net PIN1: now reaches J3.1 (Pin_1)
- net PIN1: now also U2.1 (CP1)
- net PIN10: now reaches J3.10 (Pin_10)
- net PIN10: now also U2.10 (PTA15)
- net PIN11: now reaches J3.11 (Pin_11)
- net PIN11: now also U2.11 (PTE6)
- net PIN12: now reaches J3.12 (Pin_12)
- net PIN12: now also U2.12 (PTE2)
- net TDO: now reaches J3.13 (Pin_13)
- net TDO: now also U2.13 (PTA10)
- net TDI: now reaches J3.14 (Pin_14)
- net TDI: now also U2.14 (PTC5)
- net TCK: now reaches J3.15 (Pin_15)
- net TCK: now also U2.15 (PTC4)
- net PIN16: now reaches J3.16 (Pin_16)
- net PIN16: now also U2.16 (PTA5)
- net PIN2: now reaches J3.2 (Pin_2)
- net PIN2: now also U2.2 (CP)
- net PIN3: now reaches J3.3 (Pin_3)
- net PIN3: now also U2.3 (HD)
- net PIN4: now reaches J3.4 (Pin_4)
- net PIN5: now reaches J3.5 (Pin_5)
- net PIN6: now reaches J3.6 (Pin_6)
- net PIN7: now reaches J3.7 (Pin_7)
- net PIN8: now reaches J3.8 (Pin_8)
- net PIN9: now reaches J3.9 (Pin_9)
- new net: C7.1, R6.2, Y1.1
- new net: C10.1, R7.2, Y1.2
Other:
- moved on the sheet: C2, R12, SW1
