File: mcu_power.kicad_sch (KiCad schematic)
At the start: 8 parts

Commit message: Update
Parts:
- removed C5, C6: 0.1uF, Capacitor_SMD:C_0805_2012Metric, symbol Device:C
- removed C8, C9: 10uF, Capacitor_SMD:C_0805_2012Metric, symbol Device:C
- removed L1: L, Inductor_SMD:L_0805_2012Metric, symbol Device:L
- removed R14: 0, Resistor_SMD:R_0805_2012Metric, symbol Device:R
- added U2: S32M242CCABMKHST, Package_QFP:LQFP-64-1EP_10x10mm_P0.5mm_EP6.5x6.5mm_ThermalVias, symbol MCU_NXP_S32M2:S32M242CCABMKHST
- C4: value 10uF -> 2.2uF
Connections:
- net VDD: now also U2.25 (VDD), U2.26 (VDDA), U2.9 (VDD_AE10)
- net GNDD renamed VSS
- net VSS: now also U2.28 (VSS), U2.65 (VSS)
- new net PIN27: U2.27 (VREFH)
- new net PIN4: U2.4 (BST)
- new net PIN48: U2.48 (VDDE)
- new net PIN5: U2.5 (VLS_OUT)
- new net PIN6: U2.6 (VSUP)
- new net PIN7: U2.7 (VPRE)
- new net PIN8: U2.8 (GCTL)
